File: prototypingBoards/breadboard-long-with-header.sch (EAGLE design)
At the start: 85 parts

Commit message: Cleaned up boards
Parts:
- removed PCB1, PCB2, PCB3, PCB4: PCB_DP_SQUARE-5X5, dp_pcb:PCB_DP_SQUARE-5X5
Changed lines of the file:
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@@
 <?xml version="1.0" encoding="utf-8"?>
 <!DOCTYPE eagle SYSTEM "eagle.dtd">
-<eagle version="6.5.0">
+<eagle version="7.1.0">
 <drawing>
 <settings>
@@
 <part name="TOP-2" library="p.peter-connectors" deviceset="GENERIC-1X2" device=""/>
 <part name="BOTTOM-2" library="p.peter-connectors" deviceset="GENERIC-1X2" device=""/>
-<part name="PCB1" library="dp_pcb" deviceset="PCB_DP_SQUARE" device="-5X5"/>
-<part name="PCB2" library="dp_pcb" deviceset="PCB_DP_SQUARE" device="-5X5"/>
-<part name="PCB3" library="dp_pcb" deviceset="PCB_DP_SQUARE" device="-5X5"/>
-<part name="PCB4" library="dp_pcb" deviceset="PCB_DP_SQUARE" device="-5X5"/>
 </parts>
 <sheets>
@@
 <instance part="TOP-2" gate="G$1" x="-121.92" y="43.18" rot="R270"/>
 <instance part="BOTTOM-2" gate="G$1" x="-121.92" y="20.32" rot="R270"/>
-<instance part="PCB1" gate="G$1" x="71.12" y="187.96"/>
-<instance part="PCB2" gate="G$1" x="106.68" y="187.96"/>
-<instance part="PCB3" gate="G$1" x="127" y="182.88"/>
-<instance part="PCB4" gate="G$1" x="121.92" y="162.56"/>
 </instances>
 <busses>
